File: Zmywarka.kicad_sch (KiCad schematic)
At the start: 69 parts, among them J1 Conn_01x08, Q1 BC817, Q2 BC817, Q3 BC817, Q4 BC817, SW1 SW_MEC_5G, SW2 SW_MEC_5G, SW3 SW_MEC_5G, SW4 SW_MEC_5G, U1 74HC595, U2 74HC595

Commit message: edit
Parts:
- removed SW1, SW2, SW3, SW4: SW_MEC_5G, Button_Switch_SMD:SW_Push_1P1T_NO_6x6mm_H9.5mm, symbol Switch:SW_MEC_5G
- added SW1, SW2, SW3, SW4: SW_Omron_B3FS, Button_Switch_SMD:SW_Push_1P1T_NO_6x6mm_H9.5mm, symbol Switch:SW_Omron_B3FS
Connections:
- net at U2.12 (RCLK): now also C5.2, R17.2, R18.1
- net at U2.13 (~{OE}): now also C4.2, R15.1, U1.13 (~{OE})
- net OE: now reaches R15.2
- net OE: now also J1.5 (Pin_5)
- net VCC: now reaches R21.1
- net VCC: now also R12.2, R16.2
- net at R21.2: now also SW4.2
- net at R8.2: now also U1.5 (QF)
- net at R3.2: now also U1.15 (QA)
- net at R13.1: now also J1.7 (Pin_7)
- net at R13.2: now also C2.2
- net GND: now reaches C4.1
- net GND: now also C5.1, R18.2, R20.2
- net at R6.2: now also U1.4 (QE)
- net at R14.2: now also SW2.2
- net sw_comm: now reaches R20.1
- net sw_comm: now also J1.4 (Pin_4), SW1.1, SW2.1, SW3.1, SW4.1
- net at R1.2: now also U1.2 (QC)
- net at R7.2: now also U1.6 (QG)
- net at R5.2: now also U1.3 (QD)
- net RCLK: now reaches J1.6 (Pin_6)
- net RCLK: now also R17.1
- net at U1.1 (QB): now also R2.2
- net at R16.1: now also SW3.2
- net at R12.1: now also SW1.2
Other:
- moved on the sheet: C2, C4, C5, R1, R12, R13, R14, R15, R16, R17, R18, R2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

Commit message: HD refresh
Connections:
- net GND: now also U1.8 (GND), U2.8 (GND)
- net VCC: now also U1.16 (VCC), U2.16 (VCC)
- net PLUS_DIODY: now reaches D6.2 (A)
- net at U1.7 (QH): now also R25.1
Other:
- moved on the sheet: R25
Changed lines of the file:
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@@
+    (stroke (width 0) (type default))
+  )
+  (wire (pts (xy 204.47 129.54) (xy 204.47 130.81))
     (stroke (width 0) (type default))
   )
@@
     (stroke (width 0) (type default))
   )
+  (wire (pts (xy 140.97 69.85) (xy 140.97 72.39))
+    (stroke (width 0) (type default))
+  )
   (wire (pts (xy 53.34 85.09) (xy 50.8 85.09))
     (stroke (width 0) (type default))
@@
     (stroke (width 0) (type default))
   )
+  (wire (pts (xy 140.97 105.41) (xy 140.97 107.95))
+    (stroke (width 0) (type default))
+  )
+  (wire (pts (xy 80.01 71.12) (xy 80.01 73.66))
+    (stroke (width 0) (type default))
+  )
   (wire (pts (xy 125.73 99.06) (xy 125.73 101.6))
     (stroke (width 0) (type default))
@@
     (stroke (width 0) (type default))
   )
+  (wire (pts (xy 80.01 106.68) (xy 80.01 109.22))
+    (stroke (width 0) (type default))
+  )
   (wire (pts (xy 125.73 81.28) (xy 125.73 90.17))
     (stroke (width 0) (type default))
@@
   )
   (wire (pts (xy 25.4 67.31) (xy 27.94 67.31))
+    (stroke (width 0) (type default))
+  )
+  (wire (pts (xy 90.17 96.52) (xy 93.98 96.52))
     (stroke (width 0) (type default))
   )
@@
   (label "OE" (at 113.03 73.66 180) (fields_autoplaced)
     (effects (font (size 1.27 1.27)) (justify right bottom))
+  )
+  (label "PLUS_DIODY" (at 204.47 129.54 90) (fields_autoplaced)
+    (effects (font (size 1.27 1.27)) (justify left bottom))
   )
   (label "OE" (at 151.13 44.45 270) (fields_autoplaced)
@@
     )
   )
-  (symbol (lib_id "Device:R_Small") (at 214.63 76.2 0) (unit 1)
-    (in_bom yes) (on_board yes) (dnp no) (fields_autoplaced)
-    (property "Reference" "R25" (at 217.17 76.2 0)
-      (effects (font (size 1.27 1.27)) (justify left))
-    )
-    (property "Value" "R_Small" (at 217.17 77.47 0)
-      (effects (font (size 1.27 1.27)) (justify left) hide)
-    )
-    (property "Footprint" "Resistor_SMD:R_0805_2012Metric" (at 214.63 76.2 0)
-      (effects (font (size 1.27 1.27)) hide)
-    )
-    (property "Datasheet" "~" (at 214.63 76.2 0)
-      (effects (font (size 1.27 1.27)) hide)
-    )
+  (symbol (lib_id "Device:R_Small") (at 96.52 96.52 90) (unit 1)
+    (in_bom yes) (on_board yes) (dnp no)
+    (property "Reference" "R25" (at 96.52 96.52 90)
+      (effects (font (size 1.27 1.27)))
+    )
+    (property "Value" "R_Small" (at 97.79 93.98 0)
+      (effects (font (size 1.27 1.27)) (justify left) hide)
+    )
+    (property "Footprint" "Resistor_SMD:R_0805_2012Metric" (at 96.52 96.52 0)
+      (effects (font (size 1.27 1.27)) hide)
+    )
+    (property "Datasheet" "~" (at 96.52 96.52 0)
+      (effects (font (size 1.27 1.27)) hide)
+    )

Commit message: tracking
Parts:
- removed R27, R28, R29: R_Small, Resistor_SMD:R_0805_2012Metric, symbol Device:R_Small
Connections:
- net PLUS_DIODY: no longer D6.2 (A)
- net at D16.1 (K): now also D2.1 (K), D9.1 (K), R1.1
- net digit3: now reaches D16.2 (A)
- net digit3: now also D10.2 (A), D11.2 (A), D12.2 (A), D13.2 (A), D14.2 (A), D15.2 (A)
- net OE_DIRECT: now reaches C4.2, R15.1, U1.13 (~{OE}), U2.13 (~{OE})
- net at D20.1 (K): now also D14.1 (K), D17.1 (K), D7.1 (K), R5.1
- net at R8.1: now also D10.1 (K), D23.1 (K), D3.1 (K)
- net at R3.1: now also D12.1 (K), D18.1 (K), D19.1 (K), D5.1 (K)
- net at D13.1 (K): now also D22.1 (K), D6.1 (K), R7.1
- net at D4.1 (K): now also D11.1 (K), R6.1
- net digit2: now reaches D4.2 (A)
- net digit2: now also D3.2 (A), D5.2 (A), D6.2 (A), D7.2 (A), D8.2 (A), D9.2 (A)
- net at D21.1 (K): now also R25.2
- net at D1.1 (K): now also D15.1 (K), D8.1 (K), R2.1
Other:
- moved on the sheet: D1, D10, D11, D12, D13, D14, D15, D16, D17, D18, D19, D2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

Commit message: almost done
Connections:
- net GND: now also C1.2, C2.1, C3.2, C6.1, R11.1, R23.1, R24.1, R26.2, R4.2, R9.2
- net OE_DIRECT: now also R19.2
- net VCC: now also C1.1, C3.1, C6.2, R10.2, R14.1, R19.1, R22.2, U1.10 (~{SRCLR}), U2.10 (~{SRCLR})
- net digit2: now also R9.1
- net digit3: now also R11.2
- net RCLK_DIRECT: now reaches C5.2, R17.2, R18.1, U2.12 (RCLK)
- net RCLK_DIRECT: now also U1.11 (SRCLK)
- net at U2.14 (SER): now also U1.9 (QH')
- net SER1: now reaches R4.1
- net SER1: now also C2.2, R13.2, U1.14 (SER)
- net digit1: now reaches D20.2 (A)
- net digit1: now also D1.2 (A), D19.2 (A), D2.2 (A), D23.2 (A), R24.2
- net digit4: now reaches D21.2 (A)
- net digit4: now also D17.2 (A), D18.2 (A), D22.2 (A), R26.1
Other:
- moved on the sheet: C1, C2, C3, C4, C5, C6, D1, D10, D11, D12, D13, D14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

Commit message: PCB_DONE
Parts:
- removed Q1, Q2, Q3, Q4: BC817, Package_TO_SOT_SMD:SOT-23, symbol Transistor_BJT:BC817
- added Q1, Q2, Q3, Q4: Q_PNP_BEC, Package_TO_SOT_SMD:SOT-23, symbol Device:Q_PNP_BEC
- added Q5: Q_NPN_BEC, Package_TO_SOT_SMD:SOT-23, symbol Device:Q_NPN_BEC
Connections:
- net GND: now also Q5.2 (E)
- net RCLK_DIRECT: now also Q5.1 (B)
- net VCC: now also Q1.2 (E), Q2.2 (E), Q3.2 (E), Q4.2 (E)
- net digit1: now also Q4.3 (C)
- net digit2: now also Q3.3 (C)
- net digit3: now also Q1.3 (C)
- net digit4: now also Q2.3 (C)
- net at U2.1 (QB): now also Q3.1 (B)
- net ppa: now reaches U2.11 (SRCLK)
- net ppa: now also R10.1, U1.12 (RCLK), Q5.3 (C)
- net at U2.15 (QA): now also Q1.1 (B)
- net at U2.2 (QC): now also Q2.1 (B)
- net at U2.3 (QD): now also Q4.1 (B)
Other:
- moved on the sheet: C3, R10
